Commit message: new changes1

File: rover_ws/install/my_rover/share/my_rover/urdf/imu.xacro (robot description, xacro)
@@ -1,4 +1,4 @@
 <?xml version="1.0"?>
-<robot xmlns:xacro="http://www.ros.org/wiki/xacro" name="robot">
+<robot xmlns:xacro="http://www.ros.org/wiki/xacro">
   <!-- Joint connecting the base_link to the imu_link -->
   <joint name="imu_joint" type="fixed">

File: rover_ws/install/my_rover/share/my_rover/urdf/robot.urdf.xacro (robot description, xacro)
@@ -6,4 +6,5 @@
 <xacro:include filename="gps.xacro"/>
 <xacro:include filename="imu.xacro"/>
+<xacro:include filename="cam.xacro"/>
 <xacro:property name="wheel_radius" value="0.1"/>
 <xacro:property name="wheel_length" value="0.05"/>

File: rover_ws/install/my_rover/share/my_rover/urdf/stereo.xacro (robot description, xacro)
@@ -1,52 +1,8 @@
 <?xml version="1.0"?>
 <robot xmlns:xacro="http://www.ros.org/wiki/xacro" >
-    <joint name="camera_joint" type="fixed">
-        <parent link="base_link"/>
-        <child link="camera_link"/>
-        <origin xyz="0.3 0 0.165" rpy="-0 0 0"/>
-    </joint>
-    <link name="camera_link">
-        <visual>
-            <geometry>
-            <box size="0.05 0.05 0.05"/>
-            </geometry>
-            <material name="white"/>
-        </visual>
-         <gazebo reference="camera_link">
-        <sensor type="depth" name="my_camera">
-            <update_rate>20</update_rate>
-            <visualize>true</visualize>
-            <camera name="cam">
-                <horizontal_fov>1.3962634</horizontal_fov>
-                <image>
-                    <width>640</width>
-                    <height>480</height>
-                    <format>R8B8G8</format>
-                </image>
-                <clip>
-                    <near>0.02</near>
-                    <far>300</far>
-                </clip>
-                <noise>
-                    <type>gaussian</type>
-                    <mean>0.0</mean>
-                    <stddev>0.007</stddev>
-                </noise>
-            </camera>
-            <plugin name="camera_controller" filename="libgazebo_ros_camera.so">
-                <frame_name>camera_link_optical</frame_name>
-                <min_depth>0.1</min_depth>
-                <max_depth>500</max_depth>
-            </plugin>
-        </sensor>
-    </gazebo>
-        <xacro:inertial_box mass="0.02" x="0.05" y="0.05" z="0.05">
-            <origin xyz="0.3 0 0.1" rpy="0 0 0"/>
-        </xacro:inertial_box>
-    </link>
     <joint name="stereo" type="fixed">
         <parent link="base_link"/>
         <child link="stereo_link"/>
-        <origin xyz="0.3 0 0.1" rpy="-1.57 -1.57 -1.57"/>
+        <origin xyz="0.3 0 0.165" rpy="0 0 0"/>
     </joint>
     <link name="stereo_link">
@@ -58,11 +14,12 @@
         </visual>
         <xacro:inertial_box mass="0.02" x="0.05" y="0.05" z="0.05">
-            <origin xyz="0.3 0 0.1" rpy="-1.57 -1.57 -1.57"/>
+            <origin xyz="0.3 0 0.165" rpy="0 0 0"/>
         </xacro:inertial_box>
     </link>
-    <gazebo reference="stereo_link">
+           <gazebo reference="stereo_link">
     <sensor name="camera" type="depth">
         <always_on>true</always_on>
         <update_rate>15</update_rate>
+        <visualize>true</visualize>
         <pose>0 0 0 0 0 0</pose>
         <camera name="realsense_depth_camera">
@@ -79,5 +36,5 @@
         </camera>
         <!-- https://github.com/mlherd/ros2_turtlebot3_waffle_intel_realsense -->
-        <plugin name="intel_realsense_d430_depth_driver" filename="libgazebo_ros_camera.so">
+        <plugin name="camera_controller" filename="libgazebo_ros_camera.so">
             <ros>
                 <namespace>d430</namespace>
